File: ROMDisk.kicad_pcb (KiCad board)
At the start: 2 copper layers, 85 x 65 mm, 32 parts, among them X1 Power, X2 Address, X3 Data, X4 Mode, X5 Control, X6 Clock

Commit message: Update
Parts:
- added C7: 100n, Capacitor_SMD:C_0805_2012Metric_Pad1.18x1.45mm_HandSolder, B.Cu at (133.8, 92.8)
- renumbered C9 to C1, C5 to C10, C6 to C11, C10 to C2, C1 to C3, C2 to C4, C7 to C5, C8 to C6, C3 to C8, C4 to C9, DD4 to DD1, DD5 to DD2, DD1 to DD3, DD2 to DD4, DD3 to DD5
Connections:
- net /INTE renamed /~{WRQ}
- net /Single_BCLK renamed /F2TTL
- net /Single_OSC_TTL renamed /OSC_TTL
Routing:
- net Net-(DD3-Ia=b): track 2.29 -> 4.90 mm
- net GND: vias 442 -> 543
Other:
- board text added: "~{WRQ}"
- board text removed: "INTE"
