File: ROMDisk.kicad_sch (KiCad schematic)
At the start: 29 parts, among them X1 Power, X2 Address, X3 Data, X4 Mode, X5 Control, X6 Clock

Commit message: Update
Parts:
- added C7: 100n, Capacitor_SMD:C_0805_2012Metric_Pad1.18x1.45mm_HandSolder, symbol Device:C
- renumbered C9 to C1, C5 to C10, C6 to C11, C10 to C2, C1 to C3, C2 to C4, C7 to C5, C8 to C6, C3 to C8, C4 to C9, DD4 to DD1, DD5 to DD2, DD1 to DD3, DD2 to DD4, DD3 to DD5
Connections:
- net GND: now also C7.2
- net at DD3.3 (Ia=b), R1.1: now also C7.1
- net INTE renamed ~{WRQ}
- net Single_BCLK renamed F2TTL
- net Single_OSC_TTL renamed OSC_TTL
Other:
- moved on the sheet: R1
